File: 7ch_op_amp_board_v41.brd (EAGLE design)
At the start: 10.5 x 15.2 mm, 11 parts

Commit message: Add through-hole for V+
Parts:
- added PAD9: (no value), wirepad:1,6/0,9
- PAD1, PAD2, PAD3, PAD4, PAD5, PAD6, PAD7, PAD8: device wirepad:1,6/0,8 -> wirepad:1,6/0,9
- moved PAD4 2.69 mm to (7.37, 13.7)
- moved PAD7 2.54 mm to (9.14, 13.7)
- moved PAD8 2.43 mm to (4.06, 11.6)
- moved PAD3 2.29 mm to (9.14, 11.6)
- moved PAD5 2.29 mm to (1.27, 11.6)
- moved PAD1 2.16 mm to (5.46, 13.7)
- moved PAD2 1.97 mm to (1.65, 13.7)
- moved PAD6 0.90 mm to (3.56, 13.7)
Connections:
- net V+: now also PAD9.1
Routing:
- net V-: track 13.7 -> 7.36 mm, vias 0 -> 1
- net N$23: track 8.35 -> 4.81 mm
- net N$9: track 12.2 -> 9.02 mm
- net V+: track 9.90 -> 12.6 mm
- net N$13: track 3.83 -> 6.25 mm
- net N$8: track 4.23 -> 6.64 mm
- net N$7: track 10.4 -> 8.19 mm
- net N$12: track 7.97 -> 5.88 mm
- net N$1: track 9.73 -> 7.96 mm
- net N$5: track 12.7 -> 11.4 mm
- net N$11: track 8.00 -> 9.35 mm, vias 1 -> 2
- net N$4: track 8.27 -> 6.95 mm
- net N$3: track 7.37 -> 6.40 mm
- net N$22: track 7.03 -> 6.33 mm
Other:
- board text added: "7ch v4.1"
- board text removed: "7ch v4.0"
